File: board/culticon.sch (KiCad schematic (older format))
At the start: 83 parts, among them J1 Conn_01x02, J2 Conn_01x02, J3 Conn_01x02, J4 Conn_01x02, J5 Conn_01x04, K1 SANYOU_SRD_Form_C, Q1 BT136-500, Q2 BT136-500, Q3 PN2222A, Q4 PN2222A, SW1 SW_SPST, SW2 SW_SPST, SW3 SW_SPST, T1 Transformer_1P_1S, U1 PC817, U10 RC1602A, U11 DHT11, U12 24LC64, U13 24LC64, U14 DS1307+, U15 74HC4051, U16 DHT11, U2 PC817, U3 MOC3021M, U4 MOC3021M, U5 L7805, U6 PC817, U7 PC817, U8 ATmega8-16PU, U9 74HC595, Y1 Crystal

Commit message: sch annotations
Parts:
- gave numbers to parts that had none: 4
Changed lines of the file:
@@
 	7150 2100 7250 2100
 $Comp
-L power:Earth #PWR?
+L power:Earth #PWR063
 U 1 1 5F30B515
 P 5350 7250
-F 0 "#PWR?" H 5350 7000 50  0001 C CNN
+F 0 "#PWR063" H 5350 7000 50  0001 C CNN
 F 1 "Earth" H 5350 7100 50  0001 C CNN
 F 2 "" H 5350 7250 50  0001 C CNN
@@
 $EndComp
 $Comp
-L Device:C C?
+L Device:C C14
 U 1 1 5F30AF92
 P 5250 6400
-F 0 "C?" H 5135 6354 50  0000 R CNN
+F 0 "C14" H 5135 6354 50  0000 R CNN
 F 1 "C" H 5135 6445 50  0000 R CNN
 F 2 "" H 5288 6250 50  0001 C CNN
@@
 	5250 6650 5350 6650
 $Comp
-L power:Earth #PWR?
+L power:Earth #PWR062
 U 1 1 5F345F3B
 P 5250 6250
-F 0 "#PWR?" H 5250 6000 50  0001 C CNN
+F 0 "#PWR062" H 5250 6000 50  0001 C CNN
 F 1 "Earth" H 5250 6100 50  0001 C CNN
 F 2 "" H 5250 6250 50  0001 C CNN
@@
 $EndComp
 $Comp
-L Connector_Generic:Conn_01x03 J?
+L Connector_Generic:Conn_01x03 J6
 U 1 1 5F555A0D
 P 6700 6500
-F 0 "J?" H 6700 6700 50  0000 C CNN
+F 0 "J6" H 6700 6700 50  0000 C CNN
 F 1 "Conn_01x03" H 6700 6300 50  0000 C CNN
 F 2 "" H 6700 6500 50  0001 C CNN
@@
 $EndComp
 $Comp
-L power:+5V #PWR?
+L power:+5V #PWR064
 U 1 1 5F5739E0
 P 6500 6400
-F 0 "#PWR?" H 6500 6250 50  0001 C CNN
+F 0 "#PWR064" H 6500 6250 50  0001 C CNN
 F 1 "+5V" V 6400 6500 50  0000 C CNN
 F 2 "" H 6500 6400 50  0001 C CNN
@@
 $EndComp
 $Comp
-L power:Earth #PWR?
+L power:Earth #PWR065
 U 1 1 5F574D0C
 P 6500 6600
-F 0 "#PWR?" H 6500 6350 50  0001 C CNN
+F 0 "#PWR065" H 6500 6350 50  0001 C CNN
 F 1 "Earth" H 6500 6450 50  0001 C CNN
 F 2 "" H 6500 6600 50  0001 C CNN
@@
 	6350 6650 6050 6650
 $Comp
-L Connector_Generic:Conn_01x03 J?
+L Connector_Generic:Conn_01x03 J7
 U 1 1 5F5AFBF9
 P 6700 7000
-F 0 "J?" H 6700 7200 50  0000 C CNN
+F 0 "J7" H 6700 7200 50  0000 C CNN
 F 1 "Conn_01x03" H 6700 6800 50  0000 C CNN
 F 2 "" H 6700 7000 50  0001 C CNN
@@
 $EndComp
 $Comp
-L power:+5V #PWR?
+L power:+5V #PWR066
 U 1 1 5F5AFC03
 P 6500 6900
-F 0 "#PWR?" H 6500 6750 50  0001 C CNN
+F 0 "#PWR066" H 6500 6750 50  0001 C CNN
 F 1 "+5V" V 6400 7000 50  0000 C CNN
 F 2 "" H 6500 6900 50  0001 C CNN
@@
 $EndComp
 $Comp
-L power:Earth #PWR?
+L power:Earth #PWR067
 U 1 1 5F5AFC0D
 P 6500 7100
-F 0 "#PWR?" H 6500 6850 50  0001 C CNN
+F 0 "#PWR067" H 6500 6850 50  0001 C CNN
 F 1 "Earth" H 6500 6950 50  0001 C CNN
 F 2 "" H 6500 7100 50  0001 C CNN
@@
 $EndComp
 $Comp
-L Connector_Generic:Conn_01x03 J?
+L Connector_Generic:Conn_01x03 J8
 U 1 1 5F5CF5B5
 P 6700 7500
-F 0 "J?" H 6700 7700 50  0000 C CNN
+F 0 "J8" H 6700 7700 50  0000 C CNN
 F 1 "Conn_01x03" H 6700 7300 50  0000 C CNN
 F 2 "" H 6700 7500 50  0001 C CNN
@@
 $EndComp
 $Comp
-L power:+5V #PWR?
+L power:+5V #PWR068
 U 1 1 5F5CF5BF
 P 6500 7400
-F 0 "#PWR?" H 6500 7250 50  0001 C CNN
+F 0 "#PWR068" H 6500 7250 50  0001 C CNN
 F 1 "+5V" V 6400 7500 50  0000 C CNN
 F 2 "" H 6500 7400 50  0001 C CNN
@@
 $EndComp
 $Comp
-L power:Earth #PWR?
+L power:Earth #PWR069
 U 1 1 5F5CF5C9
 P 6500 7600
-F 0 "#PWR?" H 6500 7350 50  0001 C CNN
+F 0 "#PWR069" H 6500 7350 50  0001 C CNN
 F 1 "Earth" H 6500 7450 50  0001 C CNN
 F 2 "" H 6500 7600 50  0001 C CNN
