File: board/culticon.sch (KiCad schematic (older format))
At the start: 83 parts, among them J1 Conn_01x02, J2 Conn_01x02, J3 Conn_01x02, J4 Conn_01x02, J5 Conn_01x04, J6 Conn_01x03, J7 Conn_01x03, J8 Conn_01x03, K1 SANYOU_SRD_Form_C, Q1 BT136-500, Q2 BT136-500, Q3 PN2222A, Q4 PN2222A, SW1 SW_SPST, SW2 SW_SPST, SW3 SW_SPST, T1 Transformer_1P_1S, U1 PC817, U10 RC1602A, U11 DHT11, U12 24LC64, U13 24LC64, U14 DS1307+, U15 74HC4051, U16 DHT11, U2 PC817, U3 MOC3021M, U4 MOC3021M, U5 L7805, U6 PC817, U7 PC817, U8 ATmega8-16PU, U9 74HC595, Y1 Crystal

Commit message: schem annotations
Connections:
- net LINE: now also K1.3
- net sw1_adc: no longer names the net of C13.2, R20.2, R22.1, R24.2, R25.2, U8.24 (PC1)
Other:
- note added: "..."
- note added: "EXT. COMM. (ISOLATED)"
- note added: "HOT/ALTA TENSÃO"
- note added: "PINOUT\n1- 5V (ext.)\n2- TX*\n3- RX*\n4- GND\n*(from m8)"
- note added: "SENSORS"
- note added: "ac input (110/220V)"
- note added: "dimmer1 output"
- note added: "dimmer2 output"
- note added: "place caps near ICs"
- note added: "relay output"
- moved on the sheet: C10, C11, C12, C13, C3, C4, C5, C6, C8, C9, J5, J6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

Commit message: schem tweaks & clean
Parts:
- removed TH1: NTC_5K, symbol Device:Thermistor_NTC
- C13: value 100n -> 47n
- C14: value C -> 10n
- R16: value R -> 1K
- R17: value R -> 1K 1%
- R18: value LDR -> R_PHOTO
Connections:
- net +5V: no longer R16.2
- net mux_adc: now also R16.1; no longer U15.3 (A)
- net at C13.2, R20.2, R22.1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: now also U8.25 (PC2); no longer U8.24 (PC1)
- net ldr_adc: now reaches R17.1, R18.1
- net ldr_adc: now also U8.24 (PC1); no longer U8.25 (PC2)
- net at U8.26 (PC3): no longer R16.1
- new net: R16.2, U15.3 (A)
Other:
- moved on the sheet: C13, C14, R20, R22, R24, R25, R30, R31, R32, SW1, SW2, SW3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

Commit message: pin changes
Parts:
- added C?: 10u 16V, symbol Device:CP
Connections:
- net Earth: now also C?.2
- net ldr_adc: now also U8.26 (PC3), C?.1; no longer U8.24 (PC1)
- net mux_adc: now also U8.24 (PC1); no longer U8.23 (PC0)
- net sreg_clk: now also U8.23 (PC0); no longer U8.14 (PB0)
- net sync_pulse: now also U8.14 (PB0); no longer U8.5 (PD3)
Other:
- moved on the sheet: R17, R18
Changed lines of the file:
@@
 	-1   0    0    -1
 $EndComp
-Text Label 5850 4000 0    50   ~ 0
+Text Label 5850 2300 0    50   ~ 0
 sync_pulse
 Wire Wire Line
-	5850 4000 5750 4000
+	5850 2300 5750 2300
 Text Label 5850 3900 0    50   ~ 0
 sqw_out
@@
 	5850 3800 5750 3800
 Wire Wire Line
-	5850 2300 5750 2300
+	5850 3000 5750 3000
 $Comp
 L Device:C C7
@@
 Wire Wire Line
 	3750 4050 3750 6350
-Text Label 5850 3000 0    50   ~ 0
+Text Label 5850 3100 0    50   ~ 0
 mux_adc
 Wire Wire Line
-	5850 3000 5750 3000
+	5850 3100 5750 3100
 $Comp
 L power:Earth #PWR060
@@
 Text Label 4850 6450 0    50   ~ 0
 spi_sck
-Text Label 4850 6750 0    50   ~ 0
-sreg_clk
-Text Label 5850 2300 0    50   ~ 0
+Text Label 5850 3000 0    50   ~ 0
 sreg_clk
 Wire Wire Line
@@
 $EndComp
 Wire Wire Line
-	4850 6750 4750 6750
-Wire Wire Line
 	4850 6450 4750 6450
-$Comp
-L power:+5V #PWR051
-U 1 1 604D0CF9
-P 4750 6550
-F 0 "#PWR051" H 4750 6400 50  0001 C CNN
-F 1 "+5V" V 4765 6723 50  0000 C CNN
-F 2 "" H 4750 6550 50  0001 C CNN
-F 3 "" H 4750 6550 50  0001 C CNN
-	1    4750 6550
-	0    1    -1   0
-$EndComp
 $Comp
 L power:+5V #PWR020
@@
 P 7900 2850
 F 0 "#PWR036" H 7900 2700 50  0001 C CNN
-F 1 "+5V" H 7915 3023 50  0000 C CNN
+F 1 "+5V" H 8050 2900 50  0000 C CNN
 F 2 "" H 7900 2850 50  0001 C CNN
 F 3 "" H 7900 2850 50  0001 C CNN
@@
 	5750 3200 6500 3200
 Connection ~ 6500 3200
-Text Label 5850 3100 0    50   ~ 0
+Text Label 5850 3300 0    50   ~ 0
 ldr_adc
 Wire Wire Line
-	5850 3100 5750 3100
+	5850 3300 5750 3300
 $Comp
 L Device:R_PHOTO R18
 U 1 1 6003209A
-P 8650 3400
-F 0 "R18" H 8720 3446 50  0000 L CNN
-F 1 "R_PHOTO" H 8720 3355 50  0000 L CNN
-F 2 "" V 8700 3150 50  0001 L CNN
-F 3 "~" H 8650 3350 50  0001 C CNN
-	1    8650 3400
-	1    0    0    -1
+P 7550 4800
+F 0 "R18" H 7620 4846 50  0000 L CNN
+F 1 "R_PHOTO" H 7620 4755 50  0000 L CNN
+F 2 "" V 7600 4550 50  0001 L CNN
+F 3 "~" H 7550 4750 50  0001 C CNN
+	1    7550 4800
+	-1   0    0    -1
 $EndComp
 $Comp
 L Device:R R17
 U 1 1 60032BAE
-P 8650 3000
-F 0 "R17" H 8580 2954 50  0000 R CNN
-F 1 "1K 1%" H 8580 3045 50  0000 R CNN
-F 2 "" V 8580 3000 50  0001 C CNN
-F 3 "~" H 8650 3000 50  0001 C CNN
-	1    8650 3000
+P 7850 4400
+F 0 "R17" H 7780 4354 50  0000 R CNN
+F 1 "1K 1%" H 7780 4445 50  0000 R CNN
+F 2 "" V 7780 4400 50  0001 C CNN
+F 3 "~" H 7850 4400 50  0001 C CNN
+	1    7850 4400
 	-1   0    0    1
 $EndComp
 Wire Wire Line
-	8650 3150 8650 3200
+	7850 4550 7850 4600
 $Comp
 L power:Earth #PWR029
 U 1 1 6006441F
-P 8650 3550
-F 0 "#PWR029" H 8650 3300 50  0001 C CNN
-F 1 "Earth" H 8650 3400 50  0001 C CNN
-F 2 "" H 8650 3550 50  0001 C CNN
-F 3 "~" H 8650 3550 50  0001 C CNN
-	1    8650 3550
+P 7550 4950
+F 0 "#PWR029" H 7550 4700 50  0001 C CNN
+F 1 "Earth" H 7550 4800 50  0001 C CNN
+F 2 "" H 7550 4950 50  0001 C CNN
+F 3 "~" H 7550 4950 50  0001 C CNN
+	1    7550 4950
 	-1   0    0    -1
 $EndComp
@@
 L power:+5V #PWR028
 U 1 1 60064B0E
-P 8650 2850
-F 0 "#PWR028" H 8650 2700 50  0001 C CNN
-F 1 "+5V" H 8665 3023 50  0000 C CNN
-F 2 "" H 8650 2850 50  0001 C CNN
-F 3 "" H 8650 2850 50  0001 C CNN
-	1    8650 2850
-	-1   0    0    -1
-$EndComp
-Text Label 8550 3200 2    50   ~ 0
+P 7850 4250
+F 0 "#PWR028" H 7850 4100 50  0001 C CNN
+F 1 "+5V" H 7865 4423 50  0000 C CNN
+F 2 "" H 7850 4250 50  0001 C CNN
+F 3 "" H 7850 4250 50  0001 C CNN
+	1    7850 4250
+	-1   0    0    -1
+$EndComp
+Text Label 7450 4600 2    50   ~ 0
 ldr_adc
-Wire Wire Line
-	8550 3200 8650 3200
-Connection ~ 8650 3200
-Wire Wire Line
-	8650 3200 8650 3250
+Connection ~ 7550 4600
+Wire Wire Line
+	7550 4600 7550 4650
 Wire Wire Line
 	7250 2600 7200 2600
+$Comp
+L Device:CP C?
+U 1 1 60258EBD
+P 7850 4800
+F 0 "C?" H 7968 4846 50  0000 L CNN
+F 1 "10u 16V" H 7968 4755 50  0000 L CNN
+F 2 "" H 7888 4650 50  0001 C CNN
+F 3 "~" H 7850 4800 50  0001 C CNN
+	1    7850 4800
+	1    0    0    -1
+$EndComp
+Wire Wire Line
+	7850 4600 7850 4650
+$Comp
+L power:Earth #PWR?
+U 1 1 602A620C
+P 7850 4950
+F 0 "#PWR?" H 7850 4700 50  0001 C CNN
+F 1 "Earth" H 7850 4800 50  0001 C CNN
+F 2 "" H 7850 4950 50  0001 C CNN
+F 3 "~" H 7850 4950 50  0001 C CNN
+	1    7850 4950
+	-1   0    0    -1
+$EndComp
+Wire Wire Line
+	7450 4600 7550 4600
+Wire Wire Line
+	7850 4600 7550 4600
+Connection ~ 7850 4600
+Wire Wire Line
+	4850 6750 4750 6750
+Text Label 4850 6750 0    50   ~ 0
+sreg_clk
+$Comp
+L power:+5V #PWR051
+U 1 1 604D0CF9
+P 4750 6550
+F 0 "#PWR051" H 4750 6400 50  0001 C CNN
+F 1 "+5V" V 4765 6723 50  0000 C CNN
+F 2 "" H 4750 6550 50  0001 C CNN
+F 3 "" H 4750 6550 50  0001 C CNN
+	1    4750 6550
+	0    1    -1   0
+$EndComp
 $EndSCHEMATC

Commit message: firmware cleanup & initial lcd driver sketches
Parts:
- removed C14: 10n, symbol Device:C
- removed R30, R31: R, symbol Device:R
- removed U11, U16: DHT11, Sensor:Aosong_DHT11_5.5x12.0_P2.54mm, symbol Sensor:DHT11
- R16: value 1K -> 100
Connections:
- net Earth: no longer U10.5 (R/W)
- net lcd_rs: now also U8.11 (PD5); no longer U8.12 (PD6)
- new net lcd_rw: U10.5 (R/W), U8.12 (PD6)
Changed lines of the file:
@@
 	6250 2400 6300 2400
 Wire Wire Line
-	6300 1900 6400 1900
-Wire Wire Line
-	6400 2000 6200 2000
+	6250 1900 6400 1900
+Wire Wire Line
+	6400 2000 6250 2000
 $Comp
 L power:+5V #PWR026
@@
 	0    -1   -1   0
 $EndComp
-Text Label 6200 2000 2    50   ~ 0
+Text Label 6250 2000 2    50   ~ 0
 lcd_e
 Text Label 5850 4400 0    50   ~ 0
@@
 Wire Wire Line
 	5850 4400 5750 4400
-Connection ~ 6300 2100
 Connection ~ 6300 2200
 Wire Wire Line
@@
 Wire Wire Line
 	5750 2800 6400 2800
-Wire Wire Line
-	6300 1900 6300 2100
 Connection ~ 6300 2300
 Wire Wire Line
@@
 $EndComp
 $Comp
-L power:+5V #PWR024
-U 1 1 5FC6D523
-P 5800 4700
-F 0 "#PWR024" H 5800 4550 50  0001 C CNN
-F 1 "+5V" H 5800 4850 50  0000 C CNN
-F 2 "" H 5800 4700 50  0001 C CNN
-F 3 "" H 5800 4700 50  0001 C CNN
-	1    5800 4700
-	1    0    0    -1
-$EndComp
-$Comp
-L power:Earth #PWR025
-U 1 1 5FC6D88D
-P 5800 5400
-F 0 "#PWR025" H 5800 5150 50  0001 C CNN
-F 1 "Earth" H 5800 5250 50  0001 C CNN
-F 2 "" H 5800 5400 50  0001 C CNN
-F 3 "~" H 5800 5400 50  0001 C CNN
-	1    5800 5400
-	1    0    0    -1
-$EndComp
-Wire Wire Line
-	6200 5100 6100 5100
-$Comp
 L power:Earth #PWR053
 U 1 1 6035B03C
@@
 Wire Wire Line
 	6250 1800 6400 1800
-Text Label 5850 4300 0    50   ~ 0
+Text Label 5850 4200 0    50   ~ 0
 lcd_rs
 Wire Wire Line
-	5750 4200 6200 4200
-Wire Wire Line
-	5850 4300 5750 4300
+	5850 4200 5750 4200
 Connection ~ 9250 1550
 Connection ~ 8950 1650
@@
 Text Label 7650 2600 0    50   ~ 0
 lcd_bl
-Wire Wire Line
-	6200 4200 6200 4750
-$Comp
-L Device:R R30
-U 1 1 5F327CE0
-P 6000 4750
-F 0 "R30" V 6207 4750 50  0000 C CNN
-F 1 "R" V 6116 4750 50  0000 C CNN
-F 2 "" V 5930 4750 50  0001 C CNN
-F 3 "~" H 6000 4750 50  0001 C CNN
-	1    6000 4750
-	0    1    -1   0
-$EndComp
-Wire Wire Line
-	5850 4750 5800 4750
-Wire Wire Line
-	5800 4750 5800 4700
-Wire Wire Line
-	5800 4750 5800 4800
-Connection ~ 5800 4750
-Wire Wire Line
-	6150 4750 6200 4750
-Connection ~ 6200 4750
-Wire Wire Line
-	6200 4750 6200 5100
 Text Label 5850 2800 0    50   ~ 0
 spi_sck
@@
 	5250 4900 5250 4850
 Wire Wire Line
-	3450 6550 3350 6550
-Wire Wire Line
 	4850 6250 4750 6250
 $Comp
@@
 	-1   0    0    -1
 $EndComp
-Text Label 3450 6550 0    50   ~ 0
-mux_adc
 Wire Wire Line
 	3750 6350 3950 6350
@@
 	2400 5600 2400 5650
 Wire Wire Line
-	6350 4750 6300 4750
-Wire Wire Line
-	6650 4750 6700 4750
-$Comp
-L Device:R R31
-U 1 1 5F327F41
-P 6500 4750
-F 0 "R31" V 6707 4750 50  0000 C CNN
-F 1 "R" V 6616 4750 50  0000 C CNN
-F 2 "" V 6430 4750 50  0001 C CNN
-F 3 "~" H 6500 4750 50  0001 C CNN
-	1    6500 4750
-	0    -1   -1   0
-$EndComp
-Connection ~ 6700 4750
-Wire Wire Line
-	6700 4750 6700 4800
-Wire Wire Line
-	6700 4750 6700 4700
-Wire Wire Line
-	6300 5100 6400 5100
-Wire Wire Line
-	6300 4100 5750 4100
-$Comp
-L power:Earth #PWR031
-U 1 1 601AAEB1
-P 6700 5400
-F 0 "#PWR031" H 6700 5150 50  0001 C CNN
-F 1 "Earth" H 6700 5250 50  0001 C CNN
-F 2 "" H 6700 5400 50  0001 C CNN
-F 3 "~" H 6700 5400 50  0001 C CNN
-	1    6700 5400
-	-1   0    0    -1
-$EndComp
-$Comp
-L power:+5V #PWR030
-U 1 1 601AAEA7
-P 6700 4700
-F 0 "#PWR030" H 6700 4550 50  0001 C CNN
-F 1 "+5V" H 6700 4850 50  0000 C CNN
-F 2 "" H 6700 4700 50  0001 C CNN
-F 3 "" H 6700 4700 50  0001 C CNN
-	1    6700 4700
-	-1   0    0    -1
-$EndComp
-$Comp
-L Sensor:DHT11 U11
-U 1 1 601AAE9D
-P 6700 5100
-F 0 "U11" H 6456 5146 50  0000 R CNN
-F 1 "DHT11" H 6456 5055 50  0000 R CNN
-F 2 "Sensor:Aosong_DHT11_5.5x12.0_P2.54mm" H 6700 4700 50  0001 C CNN
-F 3 "http://akizukidenshi.com/download/ds/aosong/DHT11.pdf" H 6850 5350 50  0001 C CNN
-	1    6700 5100
-	-1   0    0    -1
-$EndComp
-Wire Wire Line
-	6300 4100 6300 4750
-Connection ~ 6300 4750
-Wire Wire Line
-	6300 4750 6300 5100
-Wire Wire Line
 	4200 700  4200 750
 $Comp
@@
 Wire Wire Line
 	4200 750  4450 750
-$Comp
-L Sensor:DHT11 U16
-U 1 1 60C0C6FD
-P 5800 5100
-F 0 "U16" H 5556 5146 50  0000 R CNN
-F 1 "DHT11" H 5556 5055 50  0000 R CNN
-F 2 "Sensor:Aosong_DHT11_5.5x12.0_P2.54mm" H 5800 4700 50  0001 C CNN
-F 3 "http://akizukidenshi.com/download/ds/aosong/DHT11.pdf" H 5950 5350 50  0001 C CNN
-	1    5800 5100
-	1    0    0    -1
-$EndComp
 Connection ~ 3000 1900
 Wire Wire Line
@@
 $EndComp
 $Comp
-L Device:C C14
-U 1 1 5F30AF92
-P 3350 6350
-F 0 "C14" H 3235 6304 50  0000 R CNN
-F 1 "10n" H 3235 6395 50  0000 R CNN
-F 2 "" H 3388 6200 50  0001 C CNN
-F 3 "~" H 3350 6350 50  0001 C CNN
-	1    3350 6350
-	-1   0    0    1
-$EndComp
-Wire Wire Line
-	3350 6500 3350 6550
-Connection ~ 3350 6550
-Wire Wire Line
-	3350 6550 3300 6550
-$Comp
 L Connector_Generic:Conn_01x03 J6
 U 1 1 5F555A0D
@@
 Wire Wire Line
 	1600 1900 1600 2850
-$Comp
-L power:Earth #PWR062
-U 1 1 5F6433B4
-P 3350 6200
-F 0 "#PWR062" H 3350 5950 50  0001 C CNN
-F 1 "Earth" H 3350 6050 50  0001 C CNN
-F 2 "" H 3350 6200 50  0001 C CNN
-F 3 "~" H 3350 6200 50  0001 C CNN
-	1    3350 6200
-	-1   0    0    1
-$EndComp
 Wire Notes Line
 	550  5900 1950 5900
@@
 	7900 3200 7400 3200
 Connection ~ 7900 3200
-$Comp
-L Device:R R16
-U 1 1 5FECD341
-P 3150 6550
-F 0 "R16" V 3357 6550 50  0000 C CNN
-F 1 "1K" V 3266 6550 50  0000 C CNN
-F 2 "" V 3080 6550 50  0001 C CNN
-F 3 "~" H 3150 6550 50  0001 C CNN
-	1    3150 6550
-	0    1    -1   0
-$EndComp
-Wire Wire Line
-	3000 6550 2950 6550
 Wire Wire Line
 	5750 3200 6500 3200
@@
 	-1   0    0    -1
 $EndComp
-Text Label 7450 4600 2    50   ~ 0
-ldr_adc
 Connection ~ 7550 4600
 Wire Wire Line
@@
 	0    1    -1   0
 $EndComp
+Text Label 7450 4600 2    50   ~ 0
+ldr_adc
+Wire Wire Line
+	3000 6550 2950 6550
+Wire Wire Line
+	3300 6550 3450 6550
+Text Label 3450 6550 0    50   ~ 0
+mux_adc
+$Comp
+L Device:R R16
+U 1 1 5FECD341
+P 3150 6550
+F 0 "R16" V 3357 6550 50  0000 C CNN
+F 1 "100" V 3266 6550 50  0000 C CNN
+F 2 "" V 3080 6550 50  0001 C CNN
+F 3 "~" H 3150 6550 50  0001 C CNN
+	1    3150 6550
+	0    1    -1   0
+$EndComp
+Text Label 6250 1900 2    50   ~ 0
+lcd_rw
+Text Label 5850 4300 0    50   ~ 0
+lcd_rw
+Wire Wire Line
+	5850 4300 5750 4300
 $EndSCHEMATC

Commit message: board cleanup & optimization
Parts:
- removed C13: 47n, symbol Device:C
- removed C5, C?: 10u 16V, symbol Device:CP
- removed J5: Conn_01x04, symbol Connector_Generic:Conn_01x04
- removed J7, J8: Conn_01x03, symbol Connector_Generic:Conn_01x03
- removed Q4: PN2222A, Package_TO_SOT_THT:TO-92_Inline, symbol Transistor_BJT:PN2222A
- removed R18: R_PHOTO, symbol Device:R_PHOTO
- removed R28, R29, R9: R, symbol Device:R
- removed U6, U7: PC817, Package_DIP:DIP-4_W7.62mm, symbol Isolator:PC817
- added C5: C, symbol Device:C
- added C?: 47n, symbol Device:C
- added D3: 1N4734A, Diode_THT:D_DO-41_SOD81_P10.16mm_Horizontal, symbol Diode:1N47xxA
- added J5: ICP_Header, symbol Connector:Conn_01x06_Male
- added Q?: PN2222A, Package_TO_SOT_THT:TO-92_Inline, symbol Transistor_BJT:PN2222A
- added R18, R26, R?: 1K, symbol Device:R
- added R? (x2): 2K2, symbol Device:R
- added U6: DHT11, Sensor:Aosong_DHT11_5.5x12.0_P2.54mm, symbol Sensor:DHT11
- R1: value R -> 47K 3W
- R10, R11, R32: value R -> 220
- R12, R14, R8: value R -> 1K
- R13: value R -> 4K7
- R15: value R -> 100
- R16: value 100 -> 1K
- R17: value 1K 1% -> 1K
- RV1: value R_POT_TRIM -> 1K
Connections:
- net +5V: now also R14.1, RV1.1, U1.4, U2.4, J5.5 (Pin_5), R?.1, U6.1 (VCC); no longer R17.2, RV1.3
- net Earth: now also J6.2 (Pin_2), R16.1, R17.1, RV1.3, C5.2, C?.1, D3.2 (A), J5.1 (Pin_1), Q?.1 (E), R18.1, R26.1, R?.2, U6.4 (GND); no longer J6.3 (Pin_3), R14.2, RV1.1, U1.3, U10.10 (DB3), U10.7 (DB0), U10.8 (DB1), U10.9 (DB2), U2.3
- net lcd_e: now also U8.5 (PD3); no longer U8.13 (PD7)
- net lcd_rs: now also U8.9 (PB6/XTAL1); no longer U8.11 (PD5)
- net lcd_rw: now also U8.10 (PB7/XTAL2); no longer U8.12 (PD6)
- net mux_adc: now also R15.1; no longer R16.1
- net spi_mosi: now also J5.4 (Pin_4); no longer U10.12 (DB5)
- net spi_sck: now also J5.2 (Pin_2); no longer U10.14 (DB7)
- net sreg_clk: now also U8.16 (PB2); no longer U8.23 (PC0)
- net sync_pulse: now also Q?.3 (C), R?.2; no longer U1.4, U2.4
- net uart_rx: no longer R14.1
- net uart_tx: no longer R15.2
- net relay_t: now reaches R8.1, U9.2 (QC)
- net dim1_t: now reaches R10.1, U9.15 (QA)
- net at R20.2, R22.1, R24.2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: now also U8.23 (PC0), C?.2; no longer U8.25 (PC2)
- net dim2_t: now reaches R11.1, U9.1 (QB)
- net at R13.1, U8.1 (PC6/~RESET): now also J5.6 (Pin_6)
- net at U10.11 (DB4): now also U8.6 (PD4); no longer U8.16 (PB2)
- net at U10.13 (DB6): now also U8.12 (PD6); no longer U8.18 (PB4)
- net at R12.2: now also J6.3 (Pin_3)
- net at R12.1: now also U15.13 (A0), C5.1, D3.1 (K)
- net at R16.2: now also U10.10 (DB3); no longer U15.3 (A)
- net at U15.4 (A7): now also R14.2, U6.2 (IO)
- net ldr_adc: no longer names the net of U8.26 (PC3)
- net ldr_adc: no longer R17.1
- new net: R?.1, U1.3, U2.3
- new net: U10.12 (DB5), U8.11 (PD5)
- new net: U10.14 (DB7), U8.13 (PD7)
- new net: R26.2, U10.7 (DB0)
- new net: R18.2, U10.8 (DB1)
- new net: R17.2, U10.9 (DB2)
- new net: R15.2, U15.3 (A)
- new net: Q?.2 (B), R?.1, R?.2
- new net spi_miso: J5.3 (Pin_3), U8.18 (PB4)
Other:
- note added: "EXTERNAL SENSORS"
- note added: "mains input"
- note removed: "..."
- note removed: "EXT. COMM. (ISOLATED)"
- note removed: "PINOUT\n1- 5V (ext.)\n2- TX*\n3- RX*\n4- GND\n*(from m8)"
- note removed: "SENSORS"
- note removed: "ac input (110/220V)"
- moved on the sheet: C1, C10, C11, C12, C2, C3, C4, C6, C7, C8, C9, D1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
